File: hw/ambilight/apd_v1.0.sch (EAGLE design)
At the start: 12 parts, among them J5 POWER_JACK, Q1 220mA/50V/3.5Ω

Commit message: completed v1.0 driver
Parts:
- removed J4: (no value), SparkFun-Connectors:CONN_03JST-PTH-VERT
- removed J5: POWER_JACK, SparkFun-Connectors:POWER_JACK
- added PWR: (no value), SparkFun-Connectors:CONN_025MM
- added WS281X: (no value), SparkFun-Connectors:CONN_03POLAR
- LLC: device SparkFun-Connectors:CONN_03 -> SparkFun-Connectors:CONN_03POLAR
Connections:
- net N$1 renamed PWM_IN
- net VCC_1 renamed LVREF
- removed net N$2: J4.2, Q1.D, R2.2
- removed net VCC_2: C1.+, D1.C, J4.1, J5.PWR, LLC.3, R2.1, RPI_PWR.VBUS, SPL_PWR.VBUS
- new net 5V: C1.+, D1.A, PWR.1, RPI_PWR.VBUS, SPL_PWR.VBUS, WS281X.2
- new net HVREF: LLC.3, R2.1
- new net PWM_OUT: Q1.D, R2.2, WS281X.1
- net GND: now also PWR.2, WS281X.3; no longer J4.3, J5.GND, J5.GNDBREAK
- net N$3: now also D1.C; no longer D1.A
Other:
- moved on the sheet: D1
